File: minipad/minipad.kicad_pcb (KiCad board)
At the start: 2 copper layers, 63.5 x 44.5 mm, 23 parts, among them SW1 CherryMX_SK6812, SW2 CherryMX_SK6812, SW3 CherryMX_SK6812, SW4 CherryMX_SK6812, SW5 CherryMX_SK6812, SW6 CherryMX_SK6812, U1 RP2040-Zero

Commit message: Generated Gerber files and ordered PCBs
Other:
- board text added: "JLCJLCJLCJLC"
- board text added: "github.com/anventia made by Brendan Chen"
- board text removed: "github.com/anventia"
- board text removed: "made by Brendan Chen"
